File: PDB/power distribution board.brd (EAGLE design)
At the start: 101.6 x 30.5 mm, 11 parts

Commit message: PDB
Parts:
- moved X9 5.08 mm to (85.1, 17.8)
Routing:
- net GND: track 205.2 -> 200.1 mm
Other:
- board size 101.6 x 30.5 mm -> 96.5 x 30.5 mm
Changed lines of the file:
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@@
 <plain>
 <hole x="15.24" y="5.08" drill="3.2"/>
-<hole x="91.44" y="5.08" drill="3.2"/>
+<hole x="86.36" y="5.08" drill="3.2"/>
 <hole x="15.24" y="30.48" drill="3.2"/>
-<hole x="91.44" y="30.48" drill="3.2"/>
-<wire x1="-2.54" y1="2.54" x2="99.06" y2="2.54" width="0.4064" layer="20"/>
-<wire x1="99.06" y1="2.54" x2="99.06" y2="33.02" width="0.4064" layer="20"/>
-<wire x1="99.06" y1="33.02" x2="-2.54" y2="33.02" width="0.4064" layer="20"/>
+<hole x="86.36" y="30.48" drill="3.2"/>
+<wire x1="-2.54" y1="2.54" x2="93.98" y2="2.54" width="0.4064" layer="20"/>
+<wire x1="93.98" y1="2.54" x2="93.98" y2="33.02" width="0.4064" layer="20"/>
+<wire x1="93.98" y1="33.02" x2="-2.54" y2="33.02" width="0.4064" layer="20"/>
 <wire x1="-2.54" y1="33.02" x2="-2.54" y2="2.54" width="0.4064" layer="20"/>
 <dimension x1="-2.54" y1="2.54" x2="-2.54" y2="33.02" x3="-10.16" y3="17.78" textsize="1.778" layer="20"/>
-<dimension x1="-2.54" y1="33.02" x2="99.06" y2="33.02" x3="48.26" y3="40.64" textsize="1.778" layer="20"/>
+<dimension x1="-2.54" y1="33.02" x2="93.98" y2="33.02" x3="45.72" y3="40.64" textsize="1.778" layer="20"/>
 <dimension x1="15.24" y1="5.08" x2="15.24" y2="30.48" x3="-5.08" y3="17.78" textsize="1.778" layer="20" dtype="diameter"/>
-<dimension x1="15.24" y1="30.48" x2="91.44" y2="30.48" x3="53.34" y3="35.559996875" textsize="1.778" layer="20" dtype="diameter"/>
+<dimension x1="15.24" y1="30.48" x2="86.36" y2="30.48" x3="50.8" y3="35.559996875" textsize="1.778" layer="20" dtype="diameter"/>
 </plain>
 <attributes>
@@
 <attribute name="OC_NEWARK" value="70K9898" x="53.34" y="11.43" size="1.778" layer="27" display="off"/>
 </element>
-<element name="X9" library="con-wago-500" package="W237-4" value="" x="90.17" y="17.78" rot="R90">
-<attribute name="OC_FARNELL" value="unknown" x="90.17" y="17.78" size="1.778" layer="27" rot="R90" display="off"/>
-<attribute name="MF" value="" x="90.17" y="17.78" size="1.778" layer="27" rot="R90" display="off"/>
-<attribute name="MPN" value="" x="90.17" y="17.78" size="1.778" layer="27" rot="R90" display="off"/>
-<attribute name="OC_NEWARK" value="unknown" x="90.17" y="17.78" size="1.778" layer="27" rot="R90" display="off"/>
+<element name="X9" library="con-wago-500" package="W237-4" value="" x="85.09" y="17.78" rot="R90">
+<attribute name="OC_FARNELL" value="unknown" x="85.09" y="17.78" size="1.778" layer="27" rot="R90" display="off"/>
+<attribute name="MF" value="" x="85.09" y="17.78" size="1.778" layer="27" rot="R90" display="off"/>
+<attribute name="MPN" value="" x="85.09" y="17.78" size="1.778" layer="27" rot="R90" display="off"/>
+<attribute name="OC_NEWARK" value="unknown" x="85.09" y="17.78" size="1.778" layer="27" rot="R90" display="off"/>
 </element>
 <element name="D1" library="diode" package="DO41-10" value="1N4004" x="25.4" y="20.32"/>
@@
 <wire x1="76.16" y1="10.16" x2="76.16" y2="20.28" width="2.1844" layer="16"/>
 <wire x1="76.16" y1="20.28" x2="76.2" y2="20.32" width="2.1844" layer="16"/>
-<wire x1="76.2" y1="20.32" x2="91.44" y2="20.32" width="2.1844" layer="16"/>
-<wire x1="91.44" y1="20.32" x2="91.44" y2="25.28" width="2.1844" layer="16"/>
-<wire x1="91.44" y1="20.32" x2="91.44" y2="20.28" width="0" layer="19" extent="16-16"/>
-<wire x1="91.44" y1="10.28" x2="91.44" y2="15.28" width="2.1844" layer="16"/>
-<wire x1="91.44" y1="15.28" x2="91.44" y2="20.28" width="2.1844" layer="16"/>
+<wire x1="76.2" y1="20.32" x2="86.36" y2="20.32" width="2.1844" layer="16"/>
+<wire x1="86.36" y1="20.32" x2="86.36" y2="25.28" width="2.1844" layer="16"/>
+<wire x1="86.36" y1="10.28" x2="86.36" y2="15.28" width="2.1844" layer="16"/>
+<wire x1="86.36" y1="15.28" x2="86.36" y2="20.28" width="2.1844" layer="16"/>
 <wire x1="76.16" y1="20.28" x2="61" y2="20.28" width="2.1844" layer="16"/>
 <wire x1="61" y1="20.28" x2="60.96" y2="20.32" width="2.1844" layer="16"/>
 <wire x1="60.96" y1="20.32" x2="60.96" y2="25.36" width="2.1844" layer="16"/>
 <wire x1="60.96" y1="25.36" x2="61" y2="25.4" width="2.1844" layer="16"/>
+<wire x1="86.36" y1="20.32" x2="86.36" y2="20.28" width="2.1844" layer="16"/>
 </signal>
 <signal name="VCC">
